File: pcb/pcb.kicad_sch (KiCad schematic)
At the start: 61 parts, among them CN1 Battery, CN10 Pump_On, CN11 Pump_Drain, CN12 Battery_Cell, CN2 Bat_Sense, CN3 VBUS, CN4 3.3V, CN5 VIMM, CN6 ~{Soil_On}, CN7 Soil_Drain, CN8 Soil_Out, CN9 Water_Out, Q2 AO3401A, Q3 AO3400A, Q4 2N7002, U1 USB-C 6PIN, U2 TPS63802DLAT, U3 BQ24075RGTR, U4 TUSB320LIRWBR, U5 ESP-32S DevBoard, U6 Water_Sensor, U7 Pump

Commit message: Renamed the custom library from pcb to custom
Parts:
- U5: footprint pcb:ESP-32S_USB-C_CH340_DevBoard -> custom:ESP-32S_USB-C_CH340_DevBoard; symbol pcb:ESP-32S_USB-C_CH340_DevBoard -> custom:ESP-32S_USB-C_CH340_DevBoard
Changed lines of the file:
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@@
 	)
 	(symbol
-		(lib_id "pcb:ESP-32S_USB-C_CH340_DevBoard")
+		(lib_id "custom:ESP-32S_USB-C_CH340_DevBoard")
 		(at 223.52 72.39 0)
 		(unit 1)
@@
 			)
 		)
-		(property "Footprint" "pcb:ESP-32S_USB-C_CH340_DevBoard"
+		(property "Footprint" "custom:ESP-32S_USB-C_CH340_DevBoard"
 			(at 223.52 54.61 0)
 			(hide yes)

Commit message: Fixed some ERC issues
Parts:
- removed H1: Power_Select, EasyEDA:HDR-TH_3P-P2.54-V-M_PZ254V-11-03P, symbol EasyEDA:PZ254V-11-03P_C2937625
- renumbered CN12 to CN1, CN9 to CN10, CN10 to CN11, CN11 to CN12, CN1 to CN2, CN2 to CN3, CN3 to CN4, CN4 to CN5, CN5 to CN6, CN6 to CN7, CN7 to CN8, CN8 to CN9, L2 to L1, Q4 to Q1
Connections:
- net +3.3V: now also U5.30 (3V3)
- no-connect marks 28 -> 27
Other:
- note removed: "Power Management for +3.3V (using USB-C & Battery, with concurrent charging)"
- moved on the sheet: C1, C10, C11, C2, C3, C4, C5, C6, C7, C8, C9, CN1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

Commit message: Fully sourced all the components needed
Parts:
- removed D1: SMAJ6.0A, Diode_SMD:D_SMA, symbol Diode:SMAJ6.0A
- removed D3, D4: LED, LED_THT:LED_D4.0mm, symbol Device:LED
- removed D5: D_Schottky, Diode_SMD:D_SMA_Handsoldering, symbol Device:D_Schottky
- added D3: Schottky 40V, EasyEDA:SMA_L4.3-W2.6-LS5.2-RD, symbol EasyEDA:SMA Schottky 40V
- added D4: SMAJ6.0A, EasyEDA:SMA_L4.3-W2.6-LS5.2-RD, symbol EasyEDA:SMAJ6.0A
- added LED1: RED 2V, EasyEDA:LED-TH_BD3.0-P2.54-FD, symbol EasyEDA:LED RED 2V
- added LED2: GREEN 2V, EasyEDA:LED-TH_BD4.0-P2.54-FD, symbol EasyEDA:LED GREEN 2V
- renumbered H2 to H1
Connections:
- net +3.3V: now also D3.1
- net GND: now also D4.2
- net VBUS: now also D4.1
- net at U3.7 (#PGOOD): now also LED2.2
- net at R13.1: now also LED2.1
- net at CN12.1, Q3.3 (D), U7.1: now also D3.2
- net at R12.1: now also LED1.1
- net at U3.9 (#CHG): now also LED1.2

Commit message: Component cleanup
Parts:
- removed L1: 470nH, EasyEDA:L0805, symbol EasyEDA:0805L 470nH
- added L1: 470nH, EasyEDA:IND-SMD_L2.0-W1.6-1, symbol EasyEDA:0806L 470nH
- renumbered D4 to D1
Connections:
- net at U2.7 (L2): now also L1.1
- net at U2.9 (L1): now also L1.2
Changed lines of the file:
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@@
 		(in_pos_files yes)
 		(dnp no)
-		(property "Reference" "D4"
+		(property "Reference" "D1"
 			(at 62.484 30.9899 90)
 			(show_name no)
@@
 			(project "pcb"
 				(path "/4ed6dd03-f4d0-46d7-b0cd-4ff0bb962f04"
-					(reference "D4")
+					(reference "D1")
 					(unit 1)
 				)
@@
 	)
 	(symbol
+		(lib_id "EasyEDA:0806L 470nH")
+		(at 125.73 194.31 0)
+		(unit 1)
+		(body_style 1)
+		(exclude_from_sim no)
+		(in_bom yes)
+		(on_board yes)
+		(in_pos_files yes)
+		(dnp no)
+		(property "Reference" "L1"
+			(at 125.73 190.5 0)
+			(show_name no)
+			(do_not_autoplace no)
+			(effects
+				(font
+					(size 1.27 1.27)
+				)
+			)
+		)
+		(property "Value" "470nH"
+			(at 125.73 192.278 0)
+			(show_name no)
+			(do_not_autoplace no)
+			(effects
+				(font
+					(size 1.27 1.27)
+				)
+			)
+		)
+		(property "Footprint" "EasyEDA:IND-SMD_L2.0-W1.6-1"
+			(at 125.73 201.93 0)
+			(hide yes)
+			(show_name no)
+			(do_not_autoplace no)
+			(effects
+				(font
+					(size 1.27 1.27)
+				)
+			)
+		)
+		(property "Datasheet" "https://www.lcsc.com/datasheet/C668312.pdf"
+			(at 125.73 204.47 0)
+			(hide yes)
+			(show_name no)
+			(do_not_autoplace no)
+			(effects
+				(font
+					(size 1.27 1.27)
+				)
+			)
+		)
+		(property "Description" ""
+			(at 125.73 194.31 0)
+			(hide yes)
+			(show_name no)
+			(do_not_autoplace no)
+			(effects
+				(font
+					(size 1.27 1.27)
+				)
+			)
+		)
+		(property "Manufacturer" "muRata(村田)"
+			(at 125.73 207.01 0)
+			(hide yes)
+			(show_name no)
+			(do_not_autoplace no)
+			(effects
+				(font
+					(size 1.27 1.27)
+				)
+			)
+		)
+		(property "MPN" "DFE201612E-R47M=P2"
+			(at 125.73 209.55 0)
+			(hide yes)
+			(show_name no)
+			(do_not_autoplace no)
+			(effects
+				(font
+					(size 1.27 1.27)
+				)
+			)
+		)
+		(property "LCSC Part" "C668312"
+			(at 125.73 212.09 0)
+			(hide yes)
+			(show_name no)
+			(do_not_autoplace no)
+			(effects
+				(font
+					(size 1.27 1.27)
+				)
+			)
+		)
+		(pin "1"
+		)
+		(pin "2"
+		)
+		(instances
+			(project "pcb"
+				(path "/4ed6dd03-f4d0-46d7-b0cd-4ff0bb962f04"
+					(reference "L1")
+					(unit 1)
+				)
+			)
+		)
+	)
+	(symbol
 		(lib_id "EasyEDA:0805R 100k")
 		(at 71.12 148.59 90)
@@
 					(unit 1)
 				)
-			)
-		)
-	)
-	(symbol
-		(lib_id "EasyEDA:0805L 470nH")
-		(at 125.73 194.31 0)
-		(unit 1)
-		(body_style 1)
-		(exclude_from_sim no)
-		(in_bom yes)
-		(on_board yes)
-		(in_pos_files yes)
-		(dnp no)
-		(property "Reference" "L1"
-			(at 125.73 189.738 0)
-			(show_name no)
-			(do_not_autoplace no)
-			(effects
-				(font
-					(size 1.27 1.27)
-				)
-			)
-		)
-		(property "Value" "470nH"
-			(at 125.73 191.77 0)
-			(show_name no)
-			(do_not_autoplace no)
-			(effects
-				(font
-					(size 1.27 1.27)
-				)
-			)
-		)
-		(property "Footprint" "EasyEDA:L0805"
-			(at 125.73 201.93 0)
-			(hide yes)
-			(show_name no)
-			(do_not_autoplace no)
-			(effects
-				(font
-					(size 1.27 1.27)
-				)
-			)
-		)
-		(property "Datasheet" "https://www.lcsc.com/datasheet/C2042652.pdf"
-			(at 125.73 204.47 0)
-			(hide yes)
-			(show_name no)
-			(do_not_autoplace no)
-			(effects
-				(font
-					(size 1.27 1.27)
-				)
-			)
-		)
-		(property "Description" ""
-			(at 125.73 194.31 0)
-			(hide yes)
-			(show_name no)
-			(do_not_autoplace no)
-			(effects
-				(font
-					(size 1.27 1.27)
-				)
-			)
-		)
-		(property "Manufacturer" "muRata(村田)"
-			(at 125.73 207.01 0)
-			(hide yes)
-			(show_name no)
-			(do_not_autoplace no)
-			(effects
-				(font
-					(size 1.27 1.27)
-				)
-			)
-		)
-		(property "MPN" "LQM21PNR47MCHD"
-			(at 125.73 209.55 0)
-			(hide yes)
-			(show_name no)
-			(do_not_autoplace no)
-			(effects
-				(font
-					(size 1.27 1.27)
-				)
-			)
-		)
-		(property "LCSC Part" "C2042652"
-			(at 125.73 212.09 0)
-			(hide yes)
-			(show_name no)
-			(do_not_autoplace no)
-			(effects
-				(font
-					(size 1.27 1.27)
-				)
-			)
-		)
-		(pin "2"
-		)
-		(pin "1"
-		)
-		(instances
-			(project "pcb"
-				(path "/4ed6dd03-f4d0-46d7-b0cd-4ff0bb962f04"
-					(reference "L1")
-					(unit 1)
-				)

Commit message: Tidying up the schematic a bit
Other:
- note added: "3.3 V buck-boost regulator"
- note added: "Battery charger / power path"
- note added: "Battery: protected 1S LiPo 3.7 V nominal / 4.2 V maximum"
- note added: "ESP32 DevBoard interface"
- note added: "Pump driver"
- note added: "Soil sensor interface"
- note added: "USB-C current detection"
- note added: "USB-C power input"
- note added: "Water level input"
- note removed: "Battery: protected 1S LiPo 3.7 V nominal / 4.2 V max"
- note removed: "ESP32 Integration"
- note removed: "Soil Sensor"
- note removed: "USB-C / LiPo Battery VIMM output"
- note removed: "USB-C CC Amp Detection/Selection"
- note removed: "USB-C Power Input"
- note removed: "VIMM to +3.3V Buck-Boost"
- note removed: "Water Level Sensor"
- note removed: "Water Pump"
- title: USB-C/Battery powered ESP32 PSW (Plant Watering System) -> USB-C/Battery powered ESP32 PWS (Plant Watering System)
Changed lines of the file:
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@@
 	(paper "A3")
 	(title_block
-		(title "USB-C/Battery powered ESP32 PSW (Plant Watering System)")
+		(title "USB-C/Battery powered ESP32 PWS (Plant Watering System)")
 		(date "2026-10-03")
 		(rev "1.0")
@@
 		(end 97.79 88.9)
 		(stroke
-			(width 0.3048)
-			(type dash_dot)
+			(width 0.1524)
+			(type dash)
 			(color 0 0 0 1)
 		)
@@
 		(end 182.88 217.17)
 		(stroke
-			(width 0.3048)
-			(type dash_dot)
+			(width 0.1524)
+			(type dash)
 			(color 0 0 0 1)
 		)
@@
 		(end 270.51 148.59)
 		(stroke
-			(width 0.3048)
-			(type dash_dot)
+			(width 0.1524)
+			(type dash)
 			(color 0 0 0 1)
 		)
@@
 		(end 182.88 88.9)
 		(stroke
-			(width 0.3048)
-			(type dash_dot)
+			(width 0.1524)
+			(type dash)
 			(color 0 0 0 1)
 		)
@@
 		(end 243.84 88.9)
 		(stroke
-			(width 0.3048)
-			(type dash_dot)
+			(width 0.1524)
+			(type dash)
 			(color 0 0 0 1)
 		)
@@
 		(end 361.95 148.59)
 		(stroke
-			(width 0.3048)
-			(type dash_dot)
+			(width 0.1524)
+			(type dash)
 			(color 0 0 0 1)
 		)
@@
 	)
 	(rectangle
-		(start 247.65 20.32)
+		(start 247.65 19.05)
 		(end 292.1 88.9)
 		(stroke
-			(width 0.3048)
-			(type dash_dot)
+			(width 0.1524)
+			(type dash)
 			(color 0 0 0 1)
 		)
@@
 	)
 	(rectangle
-		(start 16.51 94.615)
+		(start 16.51 95.25)
 		(end 182.88 162.56)
 		(stroke
-			(width 0.3048)
-			(type dash_dot)
+			(width 0.1524)
+			(type dash)
 			(color 0 0 0 1)
 		)
@@
 		)
 	)
-	(rectangle
-		(start 19.05 97.536)
-		(end 53.34 105.156)
-		(stroke
-			(width 0)
-			(type solid)
-			(color 255 0 0 1)
-		)
-		(fill
-			(type color)
-			(color 255 0 15 0.4)
-		)
-	)
-	(text "USB-C Power Input"
+	(text "USB-C power input"
 		(exclude_from_sim no)
-		(at 30.226 17.272 0)
+		(at 16.51 16.51 0)
 		(effects
 			(font
@@
 				(color 0 0 0 1)
 			)
+			(justify left)
 		)
 	)
-	(text "Water Level Sensor\n"
+	(text "Water level input"
 		(exclude_from_sim no)
-		(at 261.112 17.272 0)
+		(at 247.65 16.51 0)
 		(effects
 			(font
@@
 				(color 0 0 0 1)
 			)
+			(justify left)
 		)
 	)
-	(text "USB-C CC Amp Detection/Selection"
+	(text "USB-C current detection"
 		(exclude_from_sim no)
-		(at 128.524 17.272 0)
+		(at 101.6 16.51 0)
 		(effects
 			(font
@@
 				(color 0 0 0 1)
 			)
+			(justify left)
 		)
 	)
-	(text "Battery: protected 1S LiPo \n3.7 V nominal / 4.2 V max"
+	(text "Battery: protected 1S LiPo\n3.7 V nominal / 4.2 V maximum"
 		(exclude_from_sim no)
-		(at 36.83 101.6 0)
+		(at 21.59 101.6 0)
 		(effects
 			(font
 				(size 1.27 1.27)
-				(color 255 255 255 1)
+				(color 0 0 0 1)
 			)
+			(justify left)
 		)
 	)
-	(text "Soil Sensor\n"
+	(text "Soil sensor interface"
 		(exclude_from_sim no)
-		(at 194.564 93.472 0)
+		(at 186.69 92.71 0)
 		(effects
 			(font
@@
 				(color 0 0 0 1)
 			)
+			(justify left)
 		)
 	)
-	(text "ESP32 Integration"
+	(text "ESP32 DevBoard interface"
 		(exclude_from_sim no)
-		(at 199.136 17.272 0)
+		(at 186.69 16.51 0)
 		(effects
 			(font
@@
 				(color 0 0 0 1)
 			)
+			(justify left)
 		)
 	)
-	(text "VIMM to +3.3V Buck-Boost"
+	(text "3.3 V buck-boost regulator"
 		(exclude_from_sim no)
-		(at 36.068 167.132 0)
+		(at 16.51 166.37 0)
 		(effects
 			(font
@@
 				(color 0 0 0 1)
 			)
+			(justify left)
 		)
 	)
-	(text "Water Pump\n"
+	(text "Pump driver"
 		(exclude_from_sim no)
-		(at 283.718 93.472 0)
+		(at 275.59 92.71 0)
 		(effects
 			(font
@@
 				(color 0 0 0 1)
 			)
+			(justify left)
 		)
 	)
-	(text "USB-C / LiPo Battery VIMM output"
+	(text "Battery charger / power path"
 		(exclude_from_sim no)
-		(at 41.656 92.456 0)
+		(at 16.51 92.71 0)
 		(effects
 			(font
@@
 				(color 0 0 0 1)
 			)
+			(justify left)
 		)
 	)
@@
 		(dnp no)
 		(property "Reference" "R18"
-			(at 281.94 55.88 90)
+			(at 281.94 54.61 90)
 			(show_name no)
 			(do_not_autoplace no)
@@
 		)
 		(property "Value" "1k"
-			(at 278.13 55.88 0)
+			(at 281.94 57.15 90)
 			(show_name no)
 			(do_not_autoplace no)
 			(effects
 				(font
-					(size 1.016 1.016)
+					(size 1.27 1.27)
 				)
 			)
@@
 		)
 		(property "Value" "GND"
-			(at 110.49 211.836 90)
+			(at 110.49 211.836 0)
 			(show_name no)
 			(do_not_autoplace no)
@@
 		(dnp no)
 		(property "Reference" "R20"
-			(at 309.372 134.62 90)
+			(at 309.88 133.35 90)
 			(show_name no)
 			(do_not_autoplace no)
@@
 		)
 		(property "Value" "10k"
-			(at 306.07 134.62 0)
+			(at 309.88 135.89 90)
 			(show_name no)
 			(do_not_autoplace no)
 			(effects
 				(font
-					(size 1.016 1.016)
+					(size 1.27 1.27)
 				)
 			)
@@
 		)
 		(property "Value" "+3.3V"
-			(at 215.9 30.48 90)
-			(hide yes)
+			(at 213.36 25.4 0)
 			(show_name no)
 			(do_not_autoplace no)
@@
 		(dnp no)
 		(property "Reference" "R3"
-			(at 73.914 133.35 90)
+			(at 74.93 132.08 90)
 			(show_name no)
 			(do_not_autoplace no)
@@
 		)
 		(property "Value" "100k"
-			(at 71.12 133.35 0)
+			(at 74.93 134.62 90)
 			(show_name no)
 			(do_not_autoplace no)
 			(effects
 				(font
-					(size 1.016 1.016)
+					(size 1.27 1.27)
 				)
 			)
@@
 		(dnp no)
 		(property "Reference" "R17"
-			(at 281.94 43.18 90)
+			(at 281.94 41.91 90)
 			(show_name no)
 			(do_not_autoplace no)
@@
 		)
 		(property "Value" "100k"
-			(at 278.13 43.18 0)
+			(at 281.94 44.45 90)
 			(show_name no)
 			(do_not_autoplace no)
 			(effects
 				(font
-					(size 1.016 1.016)
+					(size 1.27 1.27)
 				)
 			)
@@
 		(dnp no)
 		(property "Reference" "R2"
-			(at 72.644 200.66 90)
+			(at 66.04 199.39 90)
 			(show_name no)
 			(do_not_autoplace no)
@@
 		)
 		(property "Value" "91k"
-			(at 69.85 200.66 0)
+			(at 66.04 201.93 90)
 			(show_name no)
 			(do_not_autoplace no)
 			(effects
 				(font
-					(size 1.016 1.016)
+					(size 1.27 1.27)
 				)
 			)
@@
 		(dnp no)
 		(property "Reference" "R15"
-			(at 217.932 134.62 90)
+			(at 218.44 133.35 90)
 			(show_name no)
 			(do_not_autoplace no)
@@
 		)
 		(property "Value" "100k"
-			(at 214.63 134.62 0)
+			(at 218.44 135.89 90)
 			(show_name no)
 			(do_not_autoplace no)
 			(effects
 				(font
-					(size 1.016 1.016)
+					(size 1.27 1.27)
 				)
 			)
@@
 		(dnp no)
 		(property "Reference" "R1"
-			(at 72.644 187.96 90)
+			(at 66.04 186.69 90)
 			(show_name no)
 			(do_not_autoplace no)
@@
 		)
 		(property "Value" "511k"
-			(at 69.85 187.96 0)
+			(at 66.04 189.23 90)
 			(show_name no)
 			(do_not_autoplace no)
 			(effects
 				(font
-					(size 1.016 1.016)
+					(size 1.27 1.27)
 				)
 			)
@@
 		(dnp no)
 		(property "Reference" "R4"
-			(at 73.914 148.59 90)
+			(at 74.93 147.32 90)
 			(show_name no)
 			(do_not_autoplace no)
@@
 		)
 		(property "Value" "100k"
-			(at 71.12 148.59 0)
+			(at 74.93 149.86 90)
 			(show_name no)
 			(do_not_autoplace no)
 			(effects
 				(font
-					(size 1.016 1.016)
+					(size 1.27 1.27)
 				)
 			)
@@
 	)
 	(group ""
-		(members "88496196-3e65-417d-89aa-ab73b070c915" "f44becda-9f18-4873-83ad-95a2e3475950")
+		(members "88496196-3e65-417d-89aa-ab73b070c915")
 	)
 	(sheet_instances

Commit message: Started routing the PCB
Parts:
- removed CN10: Water_Out, EasyEDA:TESTPOINT-SMD_L3.8-W2.0_RH-5019, symbol EasyEDA:RH-5019
- removed CN11: Pump_On, EasyEDA:TESTPOINT-SMD_L3.8-W2.0_RH-5019, symbol EasyEDA:RH-5019
- removed CN12: Pump_Drain, EasyEDA:TESTPOINT-SMD_L3.8-W2.0_RH-5019, symbol EasyEDA:RH-5019
- removed CN3: Bat_Sense, EasyEDA:TESTPOINT-SMD_L3.8-W2.0_RH-5019, symbol EasyEDA:RH-5019
- removed CN4: VBUS, EasyEDA:TESTPOINT-SMD_L3.8-W2.0_RH-5019, symbol EasyEDA:RH-5019
- removed CN5: 3.3V, EasyEDA:TESTPOINT-SMD_L3.8-W2.0_RH-5019, symbol EasyEDA:RH-5019
- removed CN7: ~{Soil_On}, EasyEDA:TESTPOINT-SMD_L3.8-W2.0_RH-5019, symbol EasyEDA:RH-5019
- removed CN8: Soil_Drain, EasyEDA:TESTPOINT-SMD_L3.8-W2.0_RH-5019, symbol EasyEDA:RH-5019
- removed CN9: Soil_Out, EasyEDA:TESTPOINT-SMD_L3.8-W2.0_RH-5019, symbol EasyEDA:RH-5019
- Q1: LCSC Part C916396 -> C8545; Manufacturer JSMSEMI(杰盛微) -> JSCJ(江苏长晶)
- R1: value 511k -> 510k; symbol EasyEDA:0805R 511k -> EasyEDA:0805R 510k; LCSC Part C5159719 -> C17733; MPN FRC0805F5113TS -> 0805W8F5103T5E; Manufacturer FOJAN(富捷) -> UNI-ROYAL(Uniroyal Elec)
- R14, R16, R18: LCSC Part C95781 -> C17513; MPN RC0805FR-071KL -> 0805W8F1001T5E; Manufacturer YAGEO(国巨) -> UNI-ROYAL(Uniroyal Elec)
- R19: LCSC Part C105577 -> C17408; MPN RC0805FR-07100RL -> 0805W8F1000T5E; Manufacturer YAGEO(国巨) -> UNI-ROYAL(Uniroyal Elec)
- R2: footprint EasyEDA:R0805 -> Resistor_SMD:R_0603_1608Metric; symbol EasyEDA:0805R 91k -> EasyEDA:0603R 91k; LCSC Part C2933509 -> C23265; MPN FRC0805F9102TS -> 0603WAF9102T5E; Manufacturer FOJAN(富捷) -> UNI-ROYAL(Uniroyal Elec)
- R6: value 56.2k -> 56k; symbol EasyEDA:0805R 56.2k -> EasyEDA:0805R 56k; LCSC Part C2933471 -> C17756; MPN FRC0805F5622TS -> 0805W8F5602T5E; Manufacturer FOJAN(富捷) -> UNI-ROYAL(Uniroyal Elec)
- U4: value TUSB320LIRWBR -> TUSB320IRWBR; symbol EasyEDA:TUSB320LIRWBR -> EasyEDA:TUSB320IRWBR; LCSC Part C2836598 -> C80170; MPN TUSB320LIRWBR -> TUSB320IRWBR
Connections:
- net PUMP_ON: now also U5.20 (D21); no longer U5.22 (D18)
- net WATER_OUT: now also U5.22 (D18); no longer U5.20 (D21)
Other:
- moved on the sheet: C1, C10, C11, C3, C9, CN1, CN2, D3, R16, U7

Commit message: Finished first PCB layout
Parts:
- removed CN6: VIMM, EasyEDA:TESTPOINT-SMD_L3.8-W2.0_RH-5019, symbol EasyEDA:RH-5019
Changed lines of the file:
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@@
 	)
 	(junction
-		(at 147.32 111.76)
-		(diameter 0)
-		(color 0 0 0 0)
-	)
-	(junction
 		(at 127 111.76)
 		(diameter 0)
@@
 					(unit 1)
 				)
-			)
-		)
-	)
-	(symbol
-		(lib_id "EasyEDA:RH-5019")
-		(at 147.32 107.95 90)
-		(unit 1)
-		(body_style 1)
-		(exclude_from_sim no)
-		(in_bom yes)
-		(on_board yes)
-		(in_pos_files yes)
-		(dnp no)
-		(property "Reference" "CN6"
-			(at 147.32 100.584 90)
-			(show_name no)
-			(do_not_autoplace no)
-			(effects
-				(font
-					(size 1.27 1.27)
-				)
-			)
-		)
-		(property "Value" "VIMM"
-			(at 147.32 102.616 90)
-			(show_name no)
-			(do_not_autoplace no)
-			(effects
-				(font
-					(size 1.27 1.27)
-				)
-			)
-		)
-		(property "Footprint" "EasyEDA:TESTPOINT-SMD_L3.8-W2.0_RH-5019"
-			(at 154.94 107.95 0)
-			(hide yes)
-			(show_name no)
-			(do_not_autoplace no)
-			(effects
-				(font
-					(size 1.27 1.27)
-				)
-			)
-		)
-		(property "Datasheet" "https://www.lcsc.com/datasheet/C5199800.pdf"
-			(at 157.48 107.95 0)
-			(hide yes)
-			(show_name no)
-			(do_not_autoplace no)
-			(effects
-				(font
-					(size 1.27 1.27)
-				)
-			)
-		)
-		(property "Description" ""
-			(at 147.32 107.95 0)
-			(hide yes)
-			(show_name no)
-			(do_not_autoplace no)
-			(effects
-				(font
-					(size 1.27 1.27)
-				)
-			)
-		)
-		(property "Manufacturer" "荣和"
-			(at 160.02 107.95 0)
-			(hide yes)
-			(show_name no)
-			(do_not_autoplace no)
-			(effects
-				(font
-					(size 1.27 1.27)
-				)
-			)
-		)
-		(property "MPN" "RH-5019"
-			(at 162.56 107.95 0)
-			(hide yes)
-			(show_name no)
-			(do_not_autoplace no)
-			(effects
-				(font
-					(size 1.27 1.27)
-				)
-			)
-		)
-		(property "LCSC Part" "C5199800"
-			(at 165.1 107.95 0)
-			(hide yes)
-			(show_name no)
-			(do_not_autoplace no)
-			(effects
-				(font
-					(size 1.27 1.27)
-				)
-			)
-		)
-		(pin "1"
-		)
-		(instances
-			(project "pcb"
-				(path "/4ed6dd03-f4d0-46d7-b0cd-4ff0bb962f04"
-					(reference "CN6")
-					(unit 1)
-				)

Commit message: Lowering the cost by search for different parts (non extended ones)
Parts:
- removed CN2: Battery, EasyEDA:TESTPOINT-SMD_L3.8-W2.0_RH-5019, symbol EasyEDA:RH-5019
- C11: value 100uF -> 47uF; LCSC Part C141660 -> C16780; MPN GRM21BR60J107ME15L -> CL21A476MQYNNNE; Manufacturer muRata(村田) -> SAMSUNG(三星)
- C6: LCSC Part C29277 -> C45783; MPN CL21A226MPQNNNE -> CL21A226MAQNNNE
- D1: value SMAJ6.0A -> SMAJ5.0A; LCSC Part C223993 -> C2925443; MPN SMAJ6.0A -> SMAJ5.0A; Manufacturer Littelfuse(美国力特) -> Liown
- R7: value 1.62k -> 1.5k; LCSC Part C2933331 -> C4310; MPN FRC0805F1621TS -> 0805W8F1501T5E; Manufacturer FOJAN(富捷) -> UNI-ROYAL(厚声)
- R9: value 900k -> 910k; LCSC Part C52209984 -> C17864; MPN CL0805FN900KPS -> 0805W8F9103T5E; Manufacturer 昶龙科技 -> UNI-ROYAL(厚声)
- U4: value TUSB320IRWBR -> TUSB320LIRWBR; LCSC Part C80170 -> C2836598; MPN TUSB320IRWBR -> TUSB320LIRWBR
- renumbered C2 to C1, C1 to C2
Other:
- moved on the sheet: C3, CN1
