File: pcb/pcb.kicad_sch (KiCad schematic)
At the start: 49 parts, among them CN1 Battery_Cell, Q1 2N7002, Q2 AO3401A, Q3 AO3400A, U1 USB-C 6PIN, U2 TPS63802DLAT, U3 BQ24075RGTR, U4 TUSB320LIRWBR, U5 ESP-32S DevBoard, U6 Water_Sensor, U7 Pump

Commit message: Fixed the PCB design
Parts:
- removed C8: 100nF, EasyEDA:C0805, symbol EasyEDA:0805C 100nF
- removed D2: PESD5V0S2BT,215, EasyEDA:SOT-23_L2.9-W1.3-P1.90-LS2.4-BR, symbol EasyEDA:PESD5V0S2BT,215
- removed Q1: 2N7002, EasyEDA:SOT-23-3_L2.9-W1.3-P1.90-LS2.4-BR, symbol EasyEDA:SOT-23 2N7002
- removed R10, R11: 47k, EasyEDA:R0805, symbol EasyEDA:0805R 47k
- removed R9: 910k, EasyEDA:R0805, symbol EasyEDA:0805R 900k
- removed U4: TUSB320LIRWBR, EasyEDA:X2QFN-12_L1.6-W1.6-P0.40-TL, symbol EasyEDA:TUSB320IRWBR
- added C5: 100nF, EasyEDA:C0805, symbol EasyEDA:0805C 100nF
- added R10, R9: 5.1k, EasyEDA:R0805, symbol EasyEDA:0805R 5.1k
- C11: LCSC Part C16780 -> C141660; MPN CL21A476MQYNNNE -> GRM21BR60J107ME15L; Manufacturer SAMSUNG(三星) -> muRata(村田)
- C4: renamed from C6; LCSC Part C45783 -> C29277; MPN CL21A226MAQNNNE -> CL21A226MPQNNNE
- D1: LCSC Part C2925443 -> C223993; MPN SMAJ5.0A -> SMAJ6.0A; Manufacturer Liown -> Littelfuse(美国力特)
- R7: LCSC Part C4310 -> C2933331; MPN 0805W8F1501T5E -> FRC0805F1621TS; Manufacturer UNI-ROYAL(厚声) -> FOJAN(富捷)
- renumbered C2 to C1, C3 to C2, C5 to C3, C1 to C6, C4 to C7, C7 to C8, D3 to D2, Q2 to Q1, Q3 to Q2, R12 to R11, R13 to R12, R14 to R13, R15 to R14, R16 to R15, R17 to R16, R18 to R17, R19 to R18, R20 to R19, U2 to U1, U1 to U2, U5 to U4, U6 to U5, U7 to U6
Connections:
- net EN1 is gone; now on net VIMM: U3.6 (EN1)
- net EN2 is gone; now on net GND: U3.5 (EN2)
- net +3.3V: now also C5.1
- net GND: now also C5.2, R10.2, R9.2
- net CC1: no longer names the net of U2.A5 (CC1)
- net CC1: now also R9.1
- net CC2: no longer names the net of U2.B5 (CC2)
- net CC2: now also R10.1
- no-connect marks 27 -> 23
Other:
- note removed: "USB-C current detection"
- moved on the sheet: C1, C10, C11, C2, C3, C4, C6, C7, C8, C9, CN1, D1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

Commit message: Sourced even smaller components (and cheaper ones)
Parts:
- C1, C10, C5, C7, C9: footprint EasyEDA:C0805 -> Capacitor_SMD:C_0402_1005Metric; symbol EasyEDA:0805C 100nF -> custom:C; LCSC Part C49678 -> C1525; MPN CC0805KRX7R9BB104 -> CL05B104KO5NNNC; Manufacturer YAGEO(国巨) -> Samsung
- C11: value 47uF -> 100uF; symbol EasyEDA:0805C 100uF -> custom:C; Manufacturer muRata(村田) -> Murata
- C2, C6, C8: footprint EasyEDA:C0805 -> Capacitor_SMD:C_0603_1608Metric; symbol EasyEDA:0805C 4.7uF -> custom:C; LCSC Part C1779 -> C19666; MPN CL21A475KAQNNNE -> CL10A475KO8NNNC; Manufacturer SAMSUNG(三星) -> Samsung
- C3: footprint EasyEDA:C0805 -> Capacitor_SMD:C_0603_1608Metric; symbol EasyEDA:0805C 10uF -> custom:C; LCSC Part C440198 -> C96446; MPN GRM21BR61H106KE43L -> CL10A106MA8NRNC; Manufacturer muRata(村田) -> Samsung
- C4: footprint EasyEDA:C0805 -> Capacitor_SMD:C_0603_1608Metric; symbol EasyEDA:0805C 22uF -> custom:C; LCSC Part C29277 -> C59461; MPN CL21A226MPQNNNE -> CL10A226MQ8NRNC; Manufacturer SAMSUNG(三星) -> Samsung
- D1: value SMAJ5.0A -> SMAJ6.0A; Manufacturer Littelfuse(美国力特) -> Littelfuse
- D2: value Schottky 40V -> SS34; Manufacturer MDD(辰达半导体) -> MDD
- J1: renamed from U2; value USB-C 6PIN -> USB-C; Manufacturer hanxia(韩下) -> hanxia
- J2: renamed from CN1; value Battery_Cell -> Battery; footprint EasyEDA:CONN-TH_B2B-PH-K-S -> Connector_JST:JST_PH_S2B-PH-SM4-TB_1x02-1MP_P2.00mm_Horizontal; symbol EasyEDA:JST PH 2.0mm 1x2P -> custom:Conn_01x02; LCSC Part C5251182 -> C295747; MPN B2B-PH-K-S-GW -> S2B-PH-SM4-TB(LF)(SN)
- J3: renamed from H1; footprint EasyEDA:HDR-TH_3P-P2.54-V-M_PZ254V-11-03P -> Connector_JST:JST_PH_S3B-PH-SM4-TB_1x03-1MP_P2.00mm_Horizontal; symbol EasyEDA:PZ254V-11-03P_C2937625 -> custom:Conn_01x03; LCSC Part C2937625 -> C265101; MPN PZ254V-11-03P -> S3B-PH-SM4-TB(LF)(SN); Manufacturer XFCN(兴飞) -> JST
- J4: renamed from U6; footprint EasyEDA:CONN-TH_MX7620-7.62-02P-GN01-CU-S-A -> Connector_JST:JST_PH_S2B-PH-SM4-TB_1x02-1MP_P2.00mm_Horizontal; symbol EasyEDA:MX7620-7.62-02P-GN01-CU-S-A -> custom:Conn_01x02; LCSC Part C5188497 -> C295747; MPN MX7620-7.62-02P-GN01-Cu-S-A -> S2B-PH-SM4-TB(LF)(SN); Manufacturer MAX(迈旭) -> JST
- J5: renamed from U5; footprint EasyEDA:CONN-TH_MX7620-7.62-02P-GN01-CU-S-A -> Connector_JST:JST_PH_S2B-PH-SM4-TB_1x02-1MP_P2.00mm_Horizontal; symbol EasyEDA:MX7620-7.62-02P-GN01-CU-S-A -> custom:Conn_01x02; LCSC Part C5188497 -> C295747; MPN MX7620-7.62-02P-GN01-Cu-S-A -> S2B-PH-SM4-TB(LF)(SN); Manufacturer MAX(迈旭) -> JST
- L1: Manufacturer muRata(村田) -> Murata
- LED1: value RED 2V -> Red; footprint EasyEDA:LED-TH_BD3.0-P2.54-FD -> LED_SMD:LED_0805_2012Metric; symbol EasyEDA:LED RED 2V -> custom:LED; LCSC Part C99772 -> C84256; MPN 204-10SURD/S530-A3 -> NCD0805R1; Manufacturer EVERLIGHT(亿光) -> NationStar
- LED2: value GREEN 2V -> Green; footprint EasyEDA:LED-TH_BD4.0-P2.54-FD -> LED_SMD:LED_0805_2012Metric; symbol EasyEDA:LED GREEN 2V -> custom:LED; LCSC Part C409438 -> C2297; MPN 204-10SYGD/S530-E2 -> KT-0805G; Manufacturer EVERLIGHT(亿光) -> KENTO
- R1: footprint EasyEDA:R0805 -> Resistor_SMD:R_0402_1005Metric; symbol EasyEDA:0805R 510k -> custom:R; LCSC Part C17733 -> C11616; MPN 0805W8F5103T5E -> 0402WGF5103TCE; Manufacturer UNI-ROYAL(Uniroyal Elec) -> UNI-ROYAL
- R10, R9: footprint EasyEDA:R0805 -> Resistor_SMD:R_0402_1005Metric; symbol EasyEDA:0805R 5.1k -> custom:R; LCSC Part C27834 -> C25905; MPN 0805W8F5101T5E -> 0402WGF5101TCE; Manufacturer UNI-ROYAL(厚声) -> UNI-ROYAL
- R11, R12: footprint EasyEDA:R0805 -> Resistor_SMD:R_0402_1005Metric; symbol EasyEDA:0805R 1.5k -> custom:R; LCSC Part C4310 -> C25867; MPN 0805W8F1501T5E -> 0402WGF1501TCE; Manufacturer UNI-ROYAL(厚声) -> UNI-ROYAL
- R13, R15, R17: footprint EasyEDA:R0805 -> Resistor_SMD:R_0402_1005Metric; symbol EasyEDA:0805R 1k -> custom:R; LCSC Part C17513 -> C11702; MPN 0805W8F1001T5E -> 0402WGF1001TCE; Manufacturer UNI-ROYAL(Uniroyal Elec) -> UNI-ROYAL
- R14, R16, R3, R4: footprint EasyEDA:R0805 -> Resistor_SMD:R_0402_1005Metric; symbol EasyEDA:0805R 100k -> custom:R; LCSC Part C149504 -> C25741; MPN 0805W8F1003T5E -> 0402WGF1003TCE; Manufacturer UNI-ROYAL(厚声) -> UNI-ROYAL
- R18: footprint EasyEDA:R0805 -> Resistor_SMD:R_0402_1005Metric; symbol EasyEDA:0805R 100 -> custom:R; LCSC Part C17408 -> C25076; MPN 0805W8F1000T5E -> 0402WGF1000TCE; Manufacturer UNI-ROYAL(Uniroyal Elec) -> UNI-ROYAL
- R19, R5: footprint EasyEDA:R0805 -> Resistor_SMD:R_0402_1005Metric; symbol EasyEDA:0805R 10k -> custom:R; LCSC Part C17414 -> C25744; MPN 0805W8F1002T5E -> 0402WGF1002TCE; Manufacturer UNI-ROYAL(厚声) -> UNI-ROYAL
- R2: symbol EasyEDA:0603R 91k -> custom:R; Manufacturer UNI-ROYAL(Uniroyal Elec) -> UNI-ROYAL
- R6: footprint EasyEDA:R0805 -> Resistor_SMD:R_0402_1005Metric; symbol EasyEDA:0805R 56k -> custom:R; LCSC Part C17756 -> C25796; MPN 0805W8F5602T5E -> 0402WGF5602TCE; Manufacturer UNI-ROYAL(Uniroyal Elec) -> UNI-ROYAL
- R7: footprint EasyEDA:R0805 -> Resistor_SMD:R_0402_1005Metric; symbol EasyEDA:0805R 1.62k -> custom:R; LCSC Part C2933331 -> C25867; MPN FRC0805F1621TS -> 0402WGF1501TCE; Manufacturer FOJAN(富捷) -> UNI-ROYAL
- R8: footprint EasyEDA:R0805 -> Resistor_SMD:R_0402_1005Metric; symbol EasyEDA:0805R 2.2k -> custom:R; LCSC Part C17520 -> C25879; MPN 0805W8F2201T5E -> 0402WGF2201TCE; Manufacturer UNI-ROYAL(厚声) -> UNI-ROYAL
- U1: Manufacturer TI(德州仪器) -> Texas Instruments
- U2: renamed from U3; Manufacturer TI(德州仪器) -> Texas Instruments
- renumbered U4 to U3
Connections:
- net at R12.1: now also LED2.2; no longer LED2.1
- net at R11.1: now also LED1.2; no longer LED1.1
- net at U2.7 (#PGOOD): now also LED2.1; no longer LED2.2
- net at U2.9 (#CHG): now also LED1.1; no longer LED1.2
Other:
- moved on the sheet: C2, C9, J3, Q1, R13, R14, R15

Commit message: Added some more symbol information
Parts:
- added J6, J7: Socket_01x15, symbol custom:Socket_01x15_BOM
- C1, C10, C2, C5, C6, C7, C8, C9: JLCPCB Tier (none) -> Basic; Voltage (none) -> 16V
- C11: JLCPCB Tier (none) -> Extended; LCSC Alt (none) -> C49215609; Voltage (none) -> 6.3V
- C3: JLCPCB Tier (none) -> Basic; Voltage (none) -> 25V
- C4: JLCPCB Tier (none) -> Basic; Voltage (none) -> 6.3V
- D1, J3, L1, U2: JLCPCB Tier (none) -> Extended
- D2, LED1, LED2, Q1, Q2, R11, R12, R13, R14, R15, R16, R17: JLCPCB Tier (none) -> Basic
- J1: JLCPCB Tier (none) -> Extended; LCSC Alt (none) -> C5178532 (verify footprint)
- J2, J4, J5: JLCPCB Tier (none) -> Extended; LCSC Alt (none) -> C54582899
- R1: JLCPCB Tier (none) -> Preferred; Note (none) -> TPS63802 FB divider top: Vout = 0.5V x (1 + R1/R2) = 3.30V
- R10: JLCPCB Tier (none) -> Basic; Note (none) -> USB-C CC2 pull-down Rd (5.1k = sink, default USB power)
- R18: JLCPCB Tier (none) -> Basic; Note (none) -> Pump MOSFET gate series resistor
- R19: JLCPCB Tier (none) -> Basic; Note (none) -> Pump MOSFET gate pull-down (pump off while ESP32 boots)
- R2: JLCPCB Tier (none) -> Preferred; Note (none) -> TPS63802 FB divider bottom (see R1)
- R3: JLCPCB Tier (none) -> Basic; Note (none) -> Battery divider top, BAT_SENSE = VBAT / 2 for ESP32 ADC
- R4: JLCPCB Tier (none) -> Basic; Note (none) -> Battery divider bottom (see R3)
- R5: JLCPCB Tier (none) -> Basic; Note (none) -> BQ24075 TS: fixed 10k instead of NTC, battery temperature s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
- R6: JLCPCB Tier (none) -> Preferred; Note (none) -> BQ24075 TMR: pre-charge timer = 48 s/k x R = 45 min, fast-c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
- R7: JLCPCB Tier (none) -> Basic; Note (none) -> BQ24075 ILIM: input current limit = 1550 / R = 1.03 A
- R8: JLCPCB Tier (none) -> Basic; Note (none) -> BQ24075 ISET: fast charge current = 890 / R = 405 mA
- R9: JLCPCB Tier (none) -> Basic; Note (none) -> USB-C CC1 pull-down Rd (5.1k = sink, default USB power)
- U1: value TPS63802DLAT -> TPS63802DLAR; JLCPCB Tier (none) -> Extended; LCSC Alt (none) -> C1849531; LCSC Part C1849531 -> C2845237; MPN TPS63802DLAT -> TPS63802DLAR
- U3: now left out of the parts list
Other:
- moved on the sheet: U3

Commit message: Copied any model into the custom library to have full control of everything
Parts:
- C1, C10, C5, C7, C9: footprint Capacitor_SMD:C_0402_1005Metric -> custom:C_0402_1005Metric
- C11: footprint EasyEDA:C0805 -> custom:C_0805_2012Metric
- C2, C3, C4, C6, C8: footprint Capacitor_SMD:C_0603_1608Metric -> custom:C_0603_1608Metric
- D1: footprint EasyEDA:SMA_L4.3-W2.6-LS5.2-RD -> custom:D_SMA; symbol EasyEDA:SMAJ6.0A -> custom:D_TVS
- D2: footprint EasyEDA:SMA_L4.3-W2.6-LS5.2-RD -> custom:D_SMA; symbol EasyEDA:SMA Schottky 40V -> custom:D_Schottky
- J1: footprint EasyEDA:USB-C-SMD_HX-TYPE-C-6PIN -> custom:USB_C_Receptacle_HX_TYPE-C-6P; symbol EasyEDA:HXTYPE-C6PIN -> custom:USB_C_Receptacle_PowerOnly_6P
- J2, J4, J5: footprint Connector_JST:JST_PH_S2B-PH-SM4-TB_1x02-1MP_P2.00mm_Horizontal -> custom:JST_PH_S2B-PH-SM4-TB_1x02-1MP_P2.00mm_Horizontal
- J3: footprint Connector_JST:JST_PH_S3B-PH-SM4-TB_1x03-1MP_P2.00mm_Horizontal -> custom:JST_PH_S3B-PH-SM4-TB_1x03-1MP_P2.00mm_Horizontal
- L1: footprint EasyEDA:IND-SMD_L2.0-W1.6-1 -> custom:L_Murata_DFE201610P; symbol EasyEDA:0806L 470nH -> custom:L
- LED1, LED2: footprint LED_SMD:LED_0805_2012Metric -> custom:LED_0805_2012Metric
- Q1: footprint EasyEDA:SOT-23_L2.9-W1.3-P1.90-LS2.4-BR -> custom:SOT-23-3; symbol EasyEDA:AO3401A -> custom:AO3401A
- Q2: footprint EasyEDA:SOT-23-3_L2.9-W1.3-P1.90-LS2.4-BR -> custom:SOT-23-3; symbol EasyEDA:AO3400A -> custom:AO3400A
- R1, R10, R11, R12, R13, R14, R15, R16, R17, R18, R19, R3, R4, R5, R6, R7, R8, R9: footprint Resistor_SMD:R_0402_1005Metric -> custom:R_0402_1005Metric
- R2: footprint Resistor_SMD:R_0603_1608Metric -> custom:R_0603_1608Metric
- U1: footprint EasyEDA:VSON-10-HR_L3.0-W2.0-P0.50-BL_TI_DLA -> custom:Texas_VSON-HR-10_2x3mm_P0.5mm; symbol EasyEDA:TPS63802DLAT -> custom:TPS63802
- U2: footprint EasyEDA:QFN-16_L3.0-W3.0-P0.50-TL-EP1.7 -> custom:QFN-16-1EP_3x3mm_P0.5mm_EP1.7x1.7mm; symbol EasyEDA:BQ24075RGTR -> custom:BQ24075RGTR
Changed lines of the file:
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@@
 			)
 		)
-		(property "Footprint" "Capacitor_SMD:C_0402_1005Metric"
+		(property "Footprint" "custom:C_0402_1005Metric"
 			(at 300.99 106.68 0)
 			(hide yes)
@@
 			)
 		)
-		(property "Footprint" "Capacitor_SMD:C_0402_1005Metric"
+		(property "Footprint" "custom:C_0402_1005Metric"
 			(at 74.93 200.66 0)
 			(hide yes)
@@
 			)
 		)
-		(property "Footprint" "Capacitor_SMD:C_0603_1608Metric"
+		(property "Footprint" "custom:C_0603_1608Metric"
 			(at 77.47 182.88 0)
 			(hide yes)
@@
 	)
 	(symbol
-		(lib_id "EasyEDA:TPS63802DLAT")
+		(lib_id "custom:TPS63802")
 		(at 55.88 191.77 0)
 		(unit 1)
@@
 			)
 		)
-		(property "Footprint" "EasyEDA:VSON-10-HR_L3.0-W2.0-P0.50-BL_TI_DLA"
+		(property "Footprint" "custom:Texas_VSON-HR-10_2x3mm_P0.5mm"
 			(at 55.88 204.47 0)
 			(hide yes)
@@
 	)
 	(symbol
-		(lib_id "EasyEDA:HXTYPE-C6PIN")
+		(lib_id "custom:USB_C_Receptacle_PowerOnly_6P")
 		(at 63.5 67.31 0)
 		(unit 1)
@@
 			)
 		)
-		(property "Footprint" "EasyEDA:USB-C-SMD_HX-TYPE-C-6PIN"
+		(property "Footprint" "custom:USB_C_Receptacle_HX_TYPE-C-6P"
 			(at 63.5 91.44 0)
 			(hide yes)
@@
 			)
 		)
-		(property "Footprint" "Resistor_SMD:R_0402_1005Metric"
+		(property "Footprint" "custom:R_0402_1005Metric"
 			(at 246.38 55.88 0)
 			(hide yes)
@@
 			)
 		)
-		(property "Footprint" "Capacitor_SMD:C_0402_1005Metric"
+		(property "Footprint" "custom:C_0402_1005Metric"
 			(at 45.72 148.59 0)
 			(hide yes)
@@
 			)
 		)
-		(property "Footprint" "Capacitor_SMD:C_0402_1005Metric"
+		(property "Footprint" "custom:C_0402_1005Metric"
 			(at 214.63 115.57 0)
 			(hide yes)
@@
 			)
 		)
-		(property "Footprint" "Resistor_SMD:R_0402_1005Metric"
+		(property "Footprint" "custom:R_0402_1005Metric"
 			(at 63.5 127 0)
 			(hide yes)
@@
 			)
 		)
-		(property "Footprint" "Resistor_SMD:R_0402_1005Metric"
+		(property "Footprint" "custom:R_0402_1005Metric"
 			(at 63.5 147.32 0)
 			(hide yes)
@@
 	)
 	(symbol
-		(lib_id "EasyEDA:SMA Schottky 40V")
+		(lib_id "custom:D_Schottky")
 		(at 283.21 119.38 180)
 		(unit 1)
@@
 			)
 		)
-		(property "Footprint" "EasyEDA:SMA_L4.3-W2.6-LS5.2-RD"
+		(property "Footprint" "custom:D_SMA"
 			(at 283.21 111.76 0)
 			(hide yes)
@@
 			)
 		)
-		(property "Footprint" "Resistor_SMD:R_0402_1005Metric"
+		(property "Footprint" "custom:R_0402_1005Metric"
 			(at 121.92 132.08 0)
 			(hide yes)
@@
 			)
 		)
-		(property "Footprint" "Capacitor_SMD:C_0603_1608Metric"
+		(property "Footprint" "custom:C_0603_1608Metric"
 			(at 77.47 200.66 0)
 			(hide yes)
@@
 			)
 		)
-		(property "Footprint" "Resistor_SMD:R_0402_1005Metric"
+		(property "Footprint" "custom:R_0402_1005Metric"
 			(at 90.17 69.85 0)
 			(hide yes)
@@
 			)
 		)
-		(property "Footprint" "Resistor_SMD:R_0402_1005Metric"
+		(property "Footprint" "custom:R_0402_1005Metric"
 			(at 63.5 152.4 0)
 			(hide yes)
@@
 			)
 		)
-		(property "Footprint" "Resistor_SMD:R_0402_1005Metric"
+		(property "Footprint" "custom:R_0402_1005Metric"
 			(at 273.05 134.62 0)
 			(hide yes)
@@
 			)
 		)
-		(property "Footprint" "Capacitor_SMD:C_0603_1608Metric"
+		(property "Footprint" "custom:C_0603_1608Metric"
 			(at 43.18 123.19 0)
 			(hide yes)
@@
 			)
 		)
-		(property "Footprint" "Resistor_SMD:R_0402_1005Metric"
+		(property "Footprint" "custom:R_0402_1005Metric"
 			(at 121.92 127 0)
 			(hide yes)
@@
 			)
 		)
-		(property "Footprint" "Resistor_SMD:R_0402_1005Metric"
+		(property "Footprint" "custom:R_0402_1005Metric"
 			(at 53.34 133.35 0)
 			(hide yes)
@@
 			)
 		)
-		(property "Footprint" "LED_SMD:LED_0805_2012Metric"
+		(property "Footprint" "custom:LED_0805_2012Metric"
 			(at 111.76 133.35 0)
 			(hide yes)
@@
 			)
 		)
-		(property "Footprint" "Capacitor_SMD:C_0603_1608Metric"
+		(property "Footprint" "custom:C_0603_1608Metric"
 			(at 119.38 107.95 0)
 			(hide yes)
@@
 	)
 	(symbol
-		(lib_id "EasyEDA:SMAJ6.0A")
+		(lib_id "custom:D_TVS")
 		(at 82.55 39.37 90)
 		(unit 1)
@@
 			)
 		)
-		(property "Footprint" "EasyEDA:SMA_L4.3-W2.6-LS5.2-RD"
+		(property "Footprint" "custom:D_SMA"
 			(at 90.17 39.37 0)
 			(hide yes)
@@
 			)
 		)
-		(property "Footprint" "Resistor_SMD:R_0402_1005Metric"
+		(property "Footprint" "custom:R_0402_1005Metric"
 			(at 246.38 43.18 0)
 			(hide yes)
@@
 			)
 		)
-		(property "Footprint" "Connector_JST:JST_PH_S3B-PH-SM4-TB_1x03-1MP_P2.00mm_Horizontal"
+		(property "Footprint" "custom:JST_PH_S3B-PH-SM4-TB_1x03-1MP_P2.00mm_Horizontal"
 			(at 198.12 106.68 0)
 			(hide yes)
@@
 			)
 		)
-		(property "Footprint" "Resistor_SMD:R_0402_1005Metric"
+		(property "Footprint" "custom:R_0402_1005Metric"
 			(at 63.5 142.24 0)
 			(hide yes)
@@
 			)
 		)
-		(property "Footprint" "Resistor_SMD:R_0603_1608Metric"
+		(property "Footprint" "custom:R_0603_1608Metric"
 			(at 36.83 200.66 0)
 			(hide yes)
@@
 	)
 	(symbol
-		(lib_id "EasyEDA:BQ24075RGTR")
+		(lib_id "custom:BQ24075RGTR")
 		(at 85.09 128.27 0)
 		(unit 1)
@@
 			)
 		)
-		(property "Footprint" "EasyEDA:QFN-16_L3.0-W3.0-P0.50-TL-EP1.7"
+		(property "Footprint" "custom:QFN-16-1EP_3x3mm_P0.5mm_EP1.7x1.7mm"
 			(at 85.09 152.4 0)
 			(hide yes)
@@
 			)
 		)
-		(property "Footprint" "Resistor_SMD:R_0402_1005Metric"
+		(property "Footprint" "custom:R_0402_1005Metric"
 			(at 186.69 130.81 0)
 			(hide yes)
@@
 	)
 	(symbol
-		(lib_id "EasyEDA:AO3401A")
+		(lib_id "custom:AO3401A")
 		(at 185.42 124.46 0)
 		(unit 1)
@@
 			)
 		)
-		(property "Footprint" "EasyEDA:SOT-23_L2.9-W1.3-P1.90-LS2.4-BR"
+		(property "Footprint" "custom:SOT-23-3"
 			(at 185.42 137.16 0)
 			(hide yes)
@@
 			)
 		)
-		(property "Footprint" "Resistor_SMD:R_0402_1005Metric"
+		(property "Footprint" "custom:R_0402_1005Metric"
 			(at 36.83 187.96 0)
 			(hide yes)
@@
 			)
 		)
-		(property "Footprint" "EasyEDA:C0805"
+		(property "Footprint" "custom:C_0805_2012Metric"
 			(at 313.69 106.68 0)
 			(hide yes)
@@
 			)
 		)
-		(property "Footprint" "Resistor_SMD:R_0402_1005Metric"
+		(property "Footprint" "custom:R_0402_1005Metric"
 			(at 257.81 135.89 0)
 			(hide yes)
@@
 			)
 		)
-		(property "Footprint" "Connector_JST:JST_PH_S2B-PH-SM4-TB_1x02-1MP_P2.00mm_Horizontal"
+		(property "Footprint" "custom:JST_PH_S2B-PH-SM4-TB_1x02-1MP_P2.00mm_Horizontal"
 			(at 234.95 57.15 0)
 			(hide yes)
@@
 			)
 		)
-		(property "Footprint" "Capacitor_SMD:C_0603_1608Metric"
+		(property "Footprint" "custom:C_0603_1608Metric"
 			(at 93.98 48.26 0)
 			(hide yes)
@@
 			)
 		)
-		(property "Footprint" "LED_SMD:LED_0805_2012Metric"
+		(property "Footprint" "custom:LED_0805_2012Metric"
 			(at 111.76 128.27 0)
 			(hide yes)
@@
 	)
 	(symbol
-		(lib_id "EasyEDA:0806L 470nH")
+		(lib_id "custom:L")
 		(at 85.09 194.31 0)
 		(unit 1)
@@
 			)
 		)
-		(property "Footprint" "EasyEDA:IND-SMD_L2.0-W1.6-1"
+		(property "Footprint" "custom:L_Murata_DFE201610P"
 			(at 85.09 201.93 0)
 			(hide yes)
@@
 			)
 		)
-		(property "Footprint" "Resistor_SMD:R_0402_1005Metric"
+		(property "Footprint" "custom:R_0402_1005Metric"
 			(at 53.34 148.59 0)
 			(hide yes)
@@
 			)
 		)
-		(property "Footprint" "Connector_JST:JST_PH_S2B-PH-SM4-TB_1x02-1MP_P2.00mm_Horizontal"
+		(property "Footprint" "custom:JST_PH_S2B-PH-SM4-TB_1x02-1MP_P2.00mm_Horizontal"
 			(at 285.75 105.41 0)
 			(hide yes)
@@
 			)
 		)
-		(property "Footprint" "Connector_JST:JST_PH_S2B-PH-SM4-TB_1x02-1MP_P2.00mm_Horizontal"
+		(property "Footprint" "custom:JST_PH_S2B-PH-SM4-TB_1x02-1MP_P2.00mm_Horizontal"
 			(at 29.21 119.38 0)
 			(hide yes)
@@
 			)
 		)
-		(property "Footprint" "Capacitor_SMD:C_0402_1005Metric"
+		(property "Footprint" "custom:C_0402_1005Metric"
 			(at 106.68 48.26 0)
 			(hide yes)
@@
 			)
 		)
-		(property "Footprint" "Resistor_SMD:R_0402_1005Metric"
+		(property "Footprint" "custom:R_0402_1005Metric"
 			(at 198.12 119.38 0)
 			(hide yes)
@@
 			)
 		)
-		(property "Footprint" "Resistor_SMD:R_0402_1005Metric"
+		(property "Footprint" "custom:R_0402_1005Metric"
 			(at 90.17 72.39 0)
 			(hide yes)
@@
 			)
 		)
-		(property "Footprint" "Resistor_SMD:R_0402_1005Metric"
+		(property "Footprint" "custom:R_0402_1005Metric"
 			(at 172.72 132.08 0)
 			(hide yes)
@@
 	)
 	(symbol
-		(lib_id "EasyEDA:AO3400A")
+		(lib_id "custom:AO3400A")
 		(at 273.05 128.27 0)
 		(unit 1)
@@
 			)
 		)
-		(property "Footprint" "EasyEDA:SOT-23-3_L2.9-W1.3-P1.90-LS2.4-BR"
+		(property "Footprint" "custom:SOT-23-3"
 			(at 273.05 140.97 0)
 			(hide yes)
