File: pcb/pcb.kicad_pcb (KiCad board)
At the start: 2 copper layers, 99.7 x 99.7 mm, 60 parts, among them CN1 Battery_Cell, CN10 Water_Out, CN11 Pump_On, CN12 Pump_Drain, CN2 Battery, CN3 Bat_Sense, CN4 VBUS, CN5 3.3V, CN6 VIMM, CN7 ~{Soil_On}, CN8 Soil_Drain, CN9 Soil_Out, Q1 2N7002, Q2 AO3401A, Q3 AO3400A, U1 USB-C 6PIN, U2 TPS63802DLAT, U3 BQ24075RGTR, U4 TUSB320LIRWBR, U5 ESP-32S DevBoard, U6 Water_Sensor, U7 Pump

Commit message: Started routing the PCB
Parts:
- removed CN10: Water_Out, EasyEDA:TESTPOINT-SMD_L3.8-W2.0_RH-5019
- removed CN11: Pump_On, EasyEDA:TESTPOINT-SMD_L3.8-W2.0_RH-5019
- removed CN12: Pump_Drain, EasyEDA:TESTPOINT-SMD_L3.8-W2.0_RH-5019
- removed CN3: Bat_Sense, EasyEDA:TESTPOINT-SMD_L3.8-W2.0_RH-5019
- removed CN4: VBUS, EasyEDA:TESTPOINT-SMD_L3.8-W2.0_RH-5019
- removed CN5: 3.3V, EasyEDA:TESTPOINT-SMD_L3.8-W2.0_RH-5019
- removed CN6: VIMM, EasyEDA:TESTPOINT-SMD_L3.8-W2.0_RH-5019
- removed CN7: ~{Soil_On}, EasyEDA:TESTPOINT-SMD_L3.8-W2.0_RH-5019
- removed CN8: Soil_Drain, EasyEDA:TESTPOINT-SMD_L3.8-W2.0_RH-5019
- removed CN9: Soil_Out, EasyEDA:TESTPOINT-SMD_L3.8-W2.0_RH-5019
- R1: value 511k -> 510k
- R2: footprint EasyEDA:R0805 -> Resistor_SMD:R_0603_1608Metric
- R6: value 56.2k -> 56k
- U4: value TUSB320LIRWBR -> TUSB320IRWBR
- moved CN1 75.2 mm to (108.9, 59.3), turned to -90 degrees
- moved D3 71.7 mm to (168.7, 61.0), turned to -90 degrees
- moved CN2 65.3 mm to (117.0, 58.6), turned to 90 degrees
- moved Q2 61.5 mm to (113.0, 67.7)
- moved R15 61.5 mm to (116.7, 67.8), turned to -90 degrees
- moved C3 60.0 mm to (113.2, 58.2), turned to -90 degrees
- moved R14 57.2 mm to (119.9, 67.8), turned to -90 degrees
- moved R4 56.5 mm to (123.4, 58.1), turned to 90 degrees
- moved H1 56.4 mm to (108.9, 67.7), turned to 90 degrees
- moved R3 55.5 mm to (120.7, 58.1), turned to -90 degrees
- moved R16 53.5 mm to (124.0, 65.2), turned to 90 degrees
- moved C9 50.1 mm to (126.6, 65.3), turned to 90 degrees
- moved C2 48.4 mm to (134.9, 106.7)
- moved C8 48.2 mm to (139.1, 105.4), turned to 90 degrees
- moved R20 46.5 mm to (161.6, 63.2), turned to 90 degrees
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Connections:
- U5 pad 20: WATER_OUT -> PUMP_ON
- U5 pad 22: PUMP_ON -> WATER_OUT
Routing:
- net Net-(C3-Pad1): track 0.00 -> 71.6 mm, vias 0 -> 2
- net VBUS: track 0.00 -> 39.7 mm, vias 0 -> 2
- net +3.3V: track 0.00 -> 32.0 mm, vias 0 -> 2
- net Net-(H1-Pad3): track 0.00 -> 17.0 mm
- net VIMM: track 0.00 -> 15.1 mm
- net GND: track 0.00 -> 14.8 mm, vias 0 -> 20
- net Net-(R18-Pad1): track 0.00 -> 12.7 mm
- net ~{SOIL_ON}: track 0.00 -> 11.2 mm
- net EN1: track 0.00 -> 11.1 mm
- net BAT_SENSE: track 0.00 -> 9.74 mm
- net CC2: track 0.00 -> 8.32 mm
- net CC1: track 0.00 -> 8.26 mm
- net Net-(Q3-D): track 0.00 -> 8.25 mm
- net EN2: track 0.00 -> 6.99 mm
- net Net-(U3-ISET): track 0.00 -> 6.69 mm
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
Commit message: Finished first PCB layout
Parts:
- moved LED2 49.9 mm to (122.0, 113.0)
- moved R13 43.6 mm to (121.9, 107.6), turned to 0 degrees
- moved LED1 41.0 mm to (127.8, 113.0)
- moved R12 34.9 mm to (127.8, 107.6), turned to 0 degrees
- moved U6 0.10 mm to (173.1, 79.3)
Routing:
- net +3.3V: track 32.0 -> 152.7 mm, vias 2 -> 7
- net VIMM: track 15.1 -> 49.0 mm, vias 0 -> 2
- net Net-(U3-#PGOOD): track 0.00 -> 28.2 mm, vias 0 -> 1
- net Net-(U3-#CHG): track 0.00 -> 25.4 mm, vias 0 -> 1
- net WATER_OUT: track 3.20 -> 6.38 mm
- net Net-(LED1-Pad1): track 3.00 -> 5.59 mm
- net Net-(LED2-Pad1): track 3.46 -> 5.64 mm
- net GND: track 14.8 -> 14.5 mm, vias 20 -> 22
Other:
- board size 99.7 x 99.7 mm -> 76.7 x 66.3 mm

Commit message: Lowering the cost by search for different parts (non extended ones)
Parts:
- C11: value 100uF -> 47uF
- D1: value SMAJ6.0A -> SMAJ5.0A
- R7: value 1.62k -> 1.5k
- R9: value 900k -> 910k
- U4: value TUSB320IRWBR -> TUSB320LIRWBR
Changed lines of the file:
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@@
 			)
 		)
-		(property "Value" "1.62k"
+		(property "Value" "1.5k"
 			(at 0 4 0)
 			(layer "F.Fab")
@@
 			)
 		)
-		(property "Datasheet" "https://www.lcsc.com/datasheet/C2933331.pdf"
+		(property "Datasheet" "https://www.lcsc.com/datasheet/C4310.pdf"
 			(at 0 0 0)
 			(layer "F.Fab")
@@
 			)
 		)
-		(property "LCSC Part" "C2933331"
+		(property "LCSC Part" "C4310"
 			(at 0 0 0)
 			(layer "F.Fab")
@@
 			)
 		)
-		(property "Manufacturer" "FOJAN(富捷)"
+		(property "Manufacturer" "UNI-ROYAL(厚声)"
 			(at 0 0 180)
 			(unlocked yes)
@@
 			)
 		)
-		(property "MPN" "FRC0805F1621TS"
+		(property "MPN" "0805W8F1501T5E"
 			(at 0 0 180)
 			(unlocked yes)
@@
 			)
 		)
-		(property "Value" "900k"
+		(property "Value" "910k"
 			(at 0 4 0)
 			(layer "F.Fab")
@@
 			)
 		)
-		(property "Datasheet" "https://www.lcsc.com/datasheet/C52209984.pdf"
+		(property "Datasheet" "https://www.lcsc.com/datasheet/C17864.pdf"
 			(at 0 0 0)
 			(layer "F.Fab")
@@
 			)
 		)
-		(property "LCSC Part" "C52209984"
+		(property "LCSC Part" "C17864"
 			(at 0 0 0)
 			(layer "F.Fab")
@@
 			)
 		)
-		(property "Manufacturer" "昶龙科技"
+		(property "Manufacturer" "UNI-ROYAL(厚声)"
 			(at 0 0 180)
 			(unlocked yes)
@@
 			)
 		)
-		(property "MPN" "CL0805FN900KPS"
+		(property "MPN" "0805W8F9103T5E"
 			(at 0 0 180)
 			(unlocked yes)
@@
 			)
 		)
-		(property "Datasheet" "https://lcsc.com/product-detail/Multilayer-Ceramic-Capacitors-MLCC-SMD-SMT_SAMSUNG_CL21A226MPQNNNE_22uF-226-20-10V_C29277.html"
+		(property "Datasheet" "https://www.lcsc.com/datasheet/C45783.pdf"
 			(at 0 0 90)
 			(layer "F.Fab")
@@
 			)
 		)
-		(property "LCSC Part" "C29277"
+		(property "LCSC Part" "C45783"
 			(at 0 0 90)
 			(layer "F.Fab")
@@
 			)
 		)
-		(property "MPN" "CL21A226MPQNNNE"
+		(property "MPN" "CL21A226MAQNNNE"
 			(at 0 0 90)
 			(unlocked yes)
@@
 			)
 		)
-		(property "Value" "100uF"
+		(property "Value" "47uF"
 			(at 0 4 0)
 			(layer "F.Fab")
@@
 			)
 		)
-		(property "Datasheet" "https://lcsc.com/product-detail/Multilayer-Ceramic-Capacitors-MLCC-SMD-SMT_MuRata_GRM21BR60J107ME15L_100uF-107-20-6-3V_C141660.html"
+		(property "Datasheet" "https://www.lcsc.com/datasheet/C16780.pdf"
 			(at 0 0 0)
 			(layer "F.Fab")
@@
 			)
 		)
-		(property "LCSC Part" "C141660"
+		(property "LCSC Part" "C16780"
 			(at 0 0 0)
 			(layer "F.Fab")
@@
 			)
 		)
-		(property "Manufacturer" "muRata(村田)"
+		(property "Manufacturer" "SAMSUNG(三星)"
 			(at 0 0 180)
 			(unlocked yes)
@@
 			)
 		)
-		(property "MPN" "GRM21BR60J107ME15L"
+		(property "MPN" "CL21A476MQYNNNE"
 			(at 0 0 180)
 			(unlocked yes)
@@
 			)
 		)
-		(property "Value" "SMAJ6.0A"
+		(property "Value" "SMAJ5.0A"
 			(at 0 4 0)
 			(layer "F.Fab")
@@
 			)
 		)
-		(property "Datasheet" "https://lcsc.com/product-detail/Others_Littelfuse_SMAJ6-0A_Littelfuse-SMAJ6-0A_C223993.html"
+		(property "Datasheet" "https://www.lcsc.com/datasheet/C2925443.pdf"
 			(at 0 0 0)
 			(layer "F.Fab")
@@
 			)
 		)
-		(property "LCSC Part" "C223993"
+		(property "LCSC Part" "C2925443"
 			(at 0 0 0)
 			(layer "F.Fab")
@@
 			)
 		)
-		(property "Manufacturer" "Littelfuse(美国力特)"
+		(property "Manufacturer" "Liown"
 			(at 0 0 180)
 			(unlocked yes)
@@
 			)
 		)
-		(property "MPN" "SMAJ6.0A"
+		(property "MPN" "SMAJ5.0A"
 			(at 0 0 180)
 			(unlocked yes)
@@
 			)
 		)
-		(property "Value" "TUSB320IRWBR"
+		(property "Value" "TUSB320LIRWBR"
 			(at 0 4.75 90)
 			(layer "F.Fab")
@@
 			)
 		)
-		(property "Datasheet" "https://www.ti.com/lit/ds/symlink/tusb320.pdf"
+		(property "Datasheet" "https://www.lcsc.com/datasheet/C2836598.pdf"
 			(at 0 0 90)
 			(layer "F.Fab")
@@
 			)
 		)
-		(property "LCSC Part" "C80170"
+		(property "LCSC Part" "C2836598"
 			(at 0 0 90)
 			(layer "F.Fab")
@@
 			)
 		)
-		(property "MPN" "TUSB320IRWBR"
+		(property "MPN" "TUSB320LIRWBR"
 			(at 0 0 90)
 			(unlocked yes)

Commit message: Fixed the PCB design
Parts:
- removed the C8 at (139.1, 105.4)
- removed CN2: Battery, EasyEDA:TESTPOINT-SMD_L3.8-W2.0_RH-5019
- removed the D2 at (142.1, 109.5)
- removed the Q1 at (142.7, 101.4)
- removed the R11 at (137.0, 102.1)
- removed the U4 at (142.1, 105.5)
- added C5: 100nF, EasyEDA:C0805, F.Cu at (156.0, 108.8)
- R10: value 47k -> 5.1k
- R9: value 910k -> 5.1k
- moved R10 10.8 mm to (143.4, 108.5), turned to 90 degrees
- moved R6 6.82 mm to (143.3, 97.0), turned to -90 degrees
- moved R9 6.08 mm to (140.8, 108.5), turned to 90 degrees
- moved U3 5.65 mm to (142.1, 102.6)
- moved R5 5.06 mm to (136.4, 102.1)
- moved R8 4.30 mm to (140.9, 97.0), turned to -90 degrees
- moved R7 3.96 mm to (145.7, 97.1), turned to -90 degrees
- moved L1 2.20 mm to (149.9, 106.5)
- moved C6 1.53 mm to (136.4, 106.6)
- moved C7 1.53 mm to (136.4, 104.3)
- moved R2 1.51 mm to (151.0, 114.7), turned to 180 degrees
- moved R1 1.41 mm to (151.4, 112.7)
- moved C3 1.20 mm to (149.1, 102.7)
- moved C8 1.17 mm to (149.1, 100.3)
- moved C9 1.15 mm to (126.5, 64.1)
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- renumbered C3 to C2, C5 to C3, C6 to C4, C2 to C6, C4 to C7, C7 to C8, D3 to D2, Q2 to Q1, Q3 to Q2, R12 to R11, R13 to R12, R14 to R13, R15 to R14, R16 to R15, R17 to R16, R18 to R17, R19 to R18, R20 to R19, U2 to U1, U1 to U2, U5 to U4, U6 to U5, U7 to U6
Connections:
- R10 pad 1: +3.3V -> Net-(U2-CC2)
- R10 pad 2: EN2 -> GND
- R9 pad 1: VBUS -> Net-(U2-CC1)
- R9 pad 2: Net-(U4-VBUS_DET) -> GND
- U2 pad A5: CC1 -> Net-(U2-CC1)
- U2 pad B5: CC2 -> Net-(U2-CC2)
- U3 pad 5: EN2 -> GND
- U3 pad 6: EN1 -> VIMM
Routing:
- net +3.3V: track 152.7 -> 141.3 mm, vias 7 -> 5
- net EN1: track 11.1 -> 0.00 mm
- net CC2: track 8.32 -> 0.00 mm
- net CC1: track 8.26 -> 0.00 mm
- net Net-(C2-Pad1): track 71.6 -> 78.8 mm
- net EN2: track 6.99 -> 0.00 mm
- net VBUS: track 39.7 -> 33.0 mm
- net Net-(U3-#PGOOD): track 28.2 -> 23.5 mm
- net Net-(U3-#CHG): track 25.4 -> 21.8 mm
- net Net-(U3-ISET): track 6.69 -> 3.24 mm
- net VIMM: track 49.0 -> 52.5 mm, vias 2 -> 4
- net GND: track 14.5 -> 17.6 mm, vias 22 -> 13
- net Net-(U2-CC1): track 0.00 -> 3.07 mm
- net Net-(U2-CC2): track 0.00 -> 3.06 mm
- net Net-(U3-ILIM): track 2.44 -> 5.10 mm
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Other:
- board size 76.7 x 66.3 mm -> 77.3 x 67 mm

Commit message: Added some more symbol information
Changed lines of the file:
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@@
 			(at 0 0)
 			(size 1.5 1.5)
-			(drill 0.9)
+			(drill 1.0)
 			(layers "*.Cu" "*.Mask")
 			(remove_unused_layers yes)
@@
 			(at 0 2.54)
 			(size 1.5 1.5)
-			(drill 0.9)
+			(drill 1.0)
 			(layers "*.Cu" "*.Mask")
 			(remove_unused_layers yes)
@@
 			(at 0 5.08)
 			(size 1.5 1.5)
-			(drill 0.9)
+			(drill 1.0)
 			(layers "*.Cu" "*.Mask")
 			(remove_unused_layers yes)
@@
 			(at 0 7.62)
 			(size 1.5 1.5)
-			(drill 0.9)
+			(drill 1.0)
 			(layers "*.Cu" "*.Mask")
 			(remove_unused_layers yes)
@@
 			(at 0 10.16)
 			(size 1.5 1.5)
-			(drill 0.9)
+			(drill 1.0)
 			(layers "*.Cu" "*.Mask")
 			(remove_unused_layers yes)
@@
 			(at 0 12.7)
 			(size 1.5 1.5)
-			(drill 0.9)
+			(drill 1.0)
 			(layers "*.Cu" "*.Mask")
 			(remove_unused_layers yes)
@@
 			(at 0 15.24)
 			(size 1.5 1.5)
-			(drill 0.9)
+			(drill 1.0)
 			(layers "*.Cu" "*.Mask")
 			(remove_unused_layers yes)
@@
 			(at 0 17.78)
 			(size 1.5 1.5)
-			(drill 0.9)
+			(drill 1.0)
 			(layers "*.Cu" "*.Mask")
 			(remove_unused_layers yes)
@@
 			(at 0 20.32)
 			(size 1.5 1.5)
-			(drill 0.9)
+			(drill 1.0)
 			(layers "*.Cu" "*.Mask")
 			(remove_unused_layers yes)
@@
 			(at 0 22.86)
 			(size 1.5 1.5)
-			(drill 0.9)
+			(drill 1.0)
 			(layers "*.Cu" "*.Mask")
 			(remove_unused_layers yes)
@@
 			(at 0 25.4)
 			(size 1.5 1.5)
-			(drill 0.9)
+			(drill 1.0)
 			(layers "*.Cu" "*.Mask")
 			(remove_unused_layers yes)
@@
 			(at 0 27.94)
 			(size 1.5 1.5)
-			(drill 0.9)
+			(drill 1.0)
 			(layers "*.Cu" "*.Mask")
 			(remove_unused_layers yes)
@@
 			(at 0 30.48)
 			(size 1.5 1.5)
-			(drill 0.9)
+			(drill 1.0)
 			(layers "*.Cu" "*.Mask")
 			(remove_unused_layers yes)
@@
 			(at 0 33.02)
 			(size 1.5 1.5)
-			(drill 0.9)
+			(drill 1.0)
 			(layers "*.Cu" "*.Mask")
 			(remove_unused_layers yes)
@@
 			(at 0 35.56)
 			(size 1.5 1.5)
-			(drill 0.9)
+			(drill 1.0)
 			(layers "*.Cu" "*.Mask")
 			(remove_unused_layers yes)
@@
 			(at 25.2 0)
 			(size 1.5 1.5)
-			(drill 0.9)
+			(drill 1.0)
 			(layers "*.Cu" "*.Mask")
 			(remove_unused_layers yes)
@@
 			(at 25.2 2.54)
 			(size 1.5 1.5)
-			(drill 0.9)
+			(drill 1.0)
 			(layers "*.Cu" "*.Mask")
 			(remove_unused_layers yes)
@@
 			(at 25.2 5.08)
 			(size 1.5 1.5)
-			(drill 0.9)
+			(drill 1.0)
 			(layers "*.Cu" "*.Mask")
 			(remove_unused_layers yes)
@@
 			(at 25.2 7.62)
 			(size 1.5 1.5)
-			(drill 0.9)
+			(drill 1.0)
 			(layers "*.Cu" "*.Mask")
 			(remove_unused_layers yes)
@@
 			(at 25.2 10.16)
 			(size 1.5 1.5)
-			(drill 0.9)
+			(drill 1.0)
 			(layers "*.Cu" "*.Mask")
 			(remove_unused_layers yes)
@@
 			(at 25.2 12.7)
 			(size 1.5 1.5)
-			(drill 0.9)
+			(drill 1.0)
 			(layers "*.Cu" "*.Mask")
 			(remove_unused_layers yes)
@@
 			(at 25.2 15.24)
 			(size 1.5 1.5)
-			(drill 0.9)
+			(drill 1.0)
 			(layers "*.Cu" "*.Mask")
 			(remove_unused_layers yes)
@@
 			(at 25.2 17.78)
 			(size 1.5 1.5)
-			(drill 0.9)
+			(drill 1.0)
 			(layers "*.Cu" "*.Mask")
 			(remove_unused_layers yes)
@@
 			(at 25.2 20.32)
 			(size 1.5 1.5)
-			(drill 0.9)
+			(drill 1.0)
 			(layers "*.Cu" "*.Mask")
 			(remove_unused_layers yes)
@@
 			(at 25.2 22.86)
 			(size 1.5 1.5)
-			(drill 0.9)
+			(drill 1.0)
 			(layers "*.Cu" "*.Mask")
 			(remove_unused_layers yes)
@@
 			(at 25.2 25.4)
 			(size 1.5 1.5)
-			(drill 0.9)
+			(drill 1.0)
 			(layers "*.Cu" "*.Mask")
 			(remove_unused_layers yes)
@@
 			(at 25.2 27.94)
 			(size 1.5 1.5)
-			(drill 0.9)
+			(drill 1.0)
 			(layers "*.Cu" "*.Mask")
 			(remove_unused_layers yes)
@@
 			(at 25.2 30.48)
 			(size 1.5 1.5)
-			(drill 0.9)
+			(drill 1.0)
 			(layers "*.Cu" "*.Mask")
 			(remove_unused_layers yes)
@@
 			(at 25.2 33.02)
 			(size 1.5 1.5)
-			(drill 0.9)
+			(drill 1.0)
 			(layers "*.Cu" "*.Mask")
 			(remove_unused_layers yes)
@@
 			(at 25.2 35.56)
 			(size 1.5 1.5)
-			(drill 0.9)
-			(layers "*.Cu" "*.Mask")
-			(remove_unused_layers yes)
+			(drill 1.0)
+			(layers "*.Cu" "*.Mask")
+			(remove_unused_layers yes)
